File: digital_io.sch (KiCad schematic (older format))
At the start: 12 parts, among them Q33 NX7002AK, SW23 SW_Push, SW24 SW_Push, SW25 EC12E24204A9, SW26 EC12E24204A9

Commit message: multiple schematic and pcb changes
Parts:
- removed R35, R36, R37, R38: 10K, Resistors_SMD:R_0603, symbol R_Small
Changed lines of the file:
@@
-$EndComp
-$Comp
-L R_Small R35
-U 1 1 5A3988B1
-P 4900 4900
-F 0 "R35" H 4950 4950 50  0000 L CNN
-F 1 "10K" H 4950 4850 50  0000 L CNN
-F 2 "Resistors_SMD:R_0603" H 4900 4900 50  0001 C CNN
-F 3 "" H 4900 4900 50  0001 C CNN
-	1    4900 4900
-	1    0    0    -1
-$EndComp
-$Comp
-L +3.3V #PWR0120
-U 1 1 5A3988B8
-P 4900 4750
-F 0 "#PWR0120" H 4900 4600 50  0001 C CNN
-F 1 "+3.3V" H 4900 4890 50  0000 C CNN
-F 2 "" H 4900 4750 50  0001 C CNN
-F 3 "" H 4900 4750 50  0001 C CNN
-	1    4900 4750
-	1    0    0    -1
-$EndComp
-$Comp
-L R_Small R36
-U 1 1 5A3989A5
-P 5200 4900
-F 0 "R36" H 5250 4950 50  0000 L CNN
-F 1 "10K" H 5250 4850 50  0000 L CNN
-F 2 "Resistors_SMD:R_0603" H 5200 4900 50  0001 C CNN
-F 3 "" H 5200 4900 50  0001 C CNN
-	1    5200 4900
-	1    0    0    -1
-$EndComp
-$Comp
-L +3.3V #PWR0121
-U 1 1 5A3989AB
-P 5200 4750
-F 0 "#PWR0121" H 5200 4600 50  0001 C CNN
-F 1 "+3.3V" H 5200 4890 50  0000 C CNN
-F 2 "" H 5200 4750 50  0001 C CNN
-F 3 "" H 5200 4750 50  0001 C CNN
-	1    5200 4750
-	1    0    0    -1
 $EndComp
 $Comp
@@
 ROTARY1_B
 $Comp
-L GND #PWR0122
+L GND #PWR0120
 U 1 1 5A39D52F
 P 5700 4650
-F 0 "#PWR0122" H 5700 4400 50  0001 C CNN
+F 0 "#PWR0120" H 5700 4400 50  0001 C CNN
 F 1 "GND" H 5700 4500 50  0000 C CNN
 F 2 "" H 5700 4650 50  0001 C CNN
@@
 $EndComp
 $Comp
-L GND #PWR0123
+L GND #PWR0121
 U 1 1 5A39DA37
 P 7100 5450
-F 0 "#PWR0123" H 7100 5200 50  0001 C CNN
+F 0 "#PWR0121" H 7100 5200 50  0001 C CNN
 F 1 "GND" H 7100 5300 50  0000 C CNN
 F 2 "" H 7100 5450 50  0001 C CNN
 F 3 "" H 7100 5450 50  0001 C CNN
 	1    7100 5450
-	1    0    0    -1
-$EndComp
-$Comp
-L R_Small R37
-U 1 1 5A39DA41
-P 6800 4900
-F 0 "R37" H 6850 4950 50  0000 L CNN
-F 1 "10K" H 6850 4850 50  0000 L CNN
-F 2 "Resistors_SMD:R_0603" H 6800 4900 50  0001 C CNN
-F 3 "" H 6800 4900 50  0001 C CNN
-	1    6800 4900
-	1    0    0    -1
-$EndComp
-$Comp
-L +3.3V #PWR0124
-U 1 1 5A39DA47
-P 6800 4750
-F 0 "#PWR0124" H 6800 4600 50  0001 C CNN
-F 1 "+3.3V" H 6800 4890 50  0000 C CNN
-F 2 "" H 6800 4750 50  0001 C CNN
-F 3 "" H 6800 4750 50  0001 C CNN
-	1    6800 4750
-	1    0    0    -1
-$EndComp
-$Comp
-L R_Small R38
-U 1 1 5A39DA4E
-P 7100 4900
-F 0 "R38" H 7150 4950 50  0000 L CNN
-F 1 "10K" H 7150 4850 50  0000 L CNN
-F 2 "Resistors_SMD:R_0603" H 7100 4900 50  0001 C CNN
-F 3 "" H 7100 4900 50  0001 C CNN
-	1    7100 4900
-	1    0    0    -1
-$EndComp
-$Comp
-L +3.3V #PWR0125
-U 1 1 5A39DA54
-P 7100 4750
-F 0 "#PWR0125" H 7100 4600 50  0001 C CNN
-F 1 "+3.3V" H 7100 4890 50  0000 C CNN
-F 2 "" H 7100 4750 50  0001 C CNN
-F 3 "" H 7100 4750 50  0001 C CNN
-	1    7100 4750
 	1    0    0    -1
 $EndComp
@@
 ROTARY2_B
 $Comp
-L GND #PWR0126
+L GND #PWR0122
 U 1 1 5A39DA67
 P 7600 4650
-F 0 "#PWR0126" H 7600 4400 50  0001 C CNN
+F 0 "#PWR0122" H 7600 4400 50  0001 C CNN
 F 1 "GND" H 7600 4500 50  0000 C CNN
 F 2 "" H 7600 4650 50  0001 C CNN
@@
 $EndComp
 $Comp
-L +3.3V #PWR0127
+L +3.3V #PWR0123
 U 1 1 5A1F0C1A
 P 7050 2200
-F 0 "#PWR0127" H 7050 2050 50  0001 C CNN
+F 0 "#PWR0123" H 7050 2050 50  0001 C CNN
 F 1 "+3.3V" H 7050 2340 50  0000 C CNN
 F 2 "" H 7050 2200 50  0001 C CNN
@@
 $EndComp
 $Comp
-L GND #PWR0128
+L GND #PWR0124
 U 1 1 5A1F0FE5
 P 7050 3400
-F 0 "#PWR0128" H 7050 3150 50  0001 C CNN
+F 0 "#PWR0124" H 7050 3150 50  0001 C CNN
 F 1 "GND" H 7050 3250 50  0000 C CNN
 F 2 "" H 7050 3400 50  0001 C CNN
@@
 $EndComp
 $Comp
-L GND #PWR0129
+L GND #PWR0125
 U 1 1 5A1F45D6
 P 5700 3700
-F 0 "#PWR0129" H 5700 3450 50  0001 C CNN
+F 0 "#PWR0125" H 5700 3450 50  0001 C CNN
 F 1 "GND" H 5700 3550 50  0000 C CNN
 F 2 "" H 5700 3700 50  0001 C CNN
@@
 $EndComp
 $Comp
-L GND #PWR0130
+L GND #PWR0126
 U 1 1 5A1F45DC
 P 5200 3700
-F 0 "#PWR0130" H 5200 3450 50  0001 C CNN
+F 0 "#PWR0126" H 5200 3450 50  0001 C CNN
 F 1 "GND" H 5200 3550 50  0000 C CNN
 F 2 "" H 5200 3700 50  0001 C CNN
@@
 	4700 5150 5400 5150
 Wire Wire Line
-	4900 4750 4900 4800
-Wire Wire Line
-	5200 4750 5200 4800
-Wire Wire Line
-	5200 5000 5200 5150
-Connection ~ 5200 5150
-Wire Wire Line
-	4900 5000 4900 5350
-Connection ~ 4900 5350
-Wire Wire Line
 	4700 4150 5700 4150
 Wire Wire Line
@@
 	6600 5150 7300 5150
 Wire Wire Line
-	6800 4750 6800 4800
-Wire Wire Line
-	7100 4750 7100 4800
-Wire Wire Line
-	7100 5000 7100 5150
-Connection ~ 7100 5150
-Wire Wire Line
-	6800 5000 6800 5350
-Connection ~ 6800 5350
-Wire Wire Line
 	6600 4150 7600 4150
