File: grid.sch (KiCad schematic (older format))
At the start: 259 parts, among them Q1 BSS83P, Q10 BSS83P, Q11 BSS83P, Q12 BSS83P, Q13 BSS83P, Q14 BSS83P, Q15 BSS83P, Q16 BSS83P, Q17 BSS83P, Q18 BSS83P, Q19 BSS83P, Q2 BSS83P, Q20 BSS83P, Q21 NX7002AK, Q22 NX7002AK, Q23 NX7002AK, Q24 NX7002AK, Q25 NX7002AK, Q26 NX7002AK, Q27 NX7002AK, Q28 NX7002AK, Q29 NX7002AK, Q3 BSS83P, Q30 NX7002AK, Q31 NX7002AK, Q32 NX7002AK, Q4 BSS83P, Q5 BSS83P, Q6 BSS83P, Q7 BSS83P, Q8 BSS83P, Q9 BSS83P, SW1 Button_matrix_4x4, SW10 SW_Push, SW11 SW_Push, SW12 SW_Push, SW13 SW_Push, SW14 SW_Push, SW15 SW_Push, SW16 SW_Push, SW17 SW_Push, SW18 SW_Push, SW19 SW_Push, SW2 Button_matrix_4x4, SW20 SW_Push, SW3 Button_matrix_4x4, SW4 Button_matrix_4x4, SW5 SW_Push, SW6 SW_Push, SW7 SW_Push, SW8 SW_Push, SW9 SW_Push, U1 74HC138, U2 74HC138, U3 74HC138

Commit message: multiple schematic and pcb changes
Connections:
- net BLUE1 renamed PWM_BLUE1
- net BLUE2 renamed PWM_BLUE2
- net BLUE3 renamed PWM_BLUE3
- net BLUE4 renamed PWM_BLUE4
- net GREEN1 renamed PWM_GREEN1
- net GREEN2 renamed PWM_GREEN2
- net GREEN3 renamed PWM_GREEN3
- net GREEN4 renamed PWM_GREEN4
- net RED1 renamed PWM_RED1
- net RED2 renamed PWM_RED2
- net RED3 renamed PWM_RED3
- net RED4 renamed PWM_RED4

Commit message: pcb in development
Connections:
- net GRID_BUTTON4: now reaches D100.1 (K), D102.1 (K), D104.1 (K), D130.1 (K), D131.1 (K), D143.1 (K), D145.1 (K), D2.1 (K), D34.1 (K), D36.1 (K), D38.1 (K), D4.1 (K), D40.1 (K), D6.1 (K), D66.1 (K), D68.1 (K), D70.1 (K), D72.1 (K), D8.1 (K), D98.1 (K)
- net BUTTON1 renamed GRID_BUTTON1
- net BUTTON2 renamed GRID_BUTTON2
- net BUTTON3 renamed GRID_BUTTON3
Changed lines of the file:
@@
 PWM_BLUE4
 Text Label 4500 4700 0    60   ~ 0
-BUTTON1
+GRID_BUTTON1
 Text Label 4500 4600 0    60   ~ 0
-BUTTON2
+GRID_BUTTON2
 Text Label 4500 4500 0    60   ~ 0
-BUTTON3
+GRID_BUTTON3
 Text Label 4500 4400 0    60   ~ 0
-BUTTON4
+GRID_BUTTON4
 Entry Wire Line
 	4300 4300 4400 4400
@@
 	4300 4600 4400 4700
 Text HLabel 1800 4300 0    60   Output ~ 0
-BUTTON[1..4]
+GRID_BUTTON[1..4]
 Text HLabel 1800 6400 0    60   Input ~ 0
 PWM_RED[1..4]
@@
 $EndComp
 Text Label 1850 4300 0    60   ~ 0
-BUTTON[1..4]
+GRID_BUTTON[1..4]
 Text Label 1850 6400 0    60   ~ 0
 PWM_RED[1..4]
@@
 	1    0    0    -1
 $EndComp
+Connection ~ 6050 4400
 $EndSCHEMATC

Commit message: commiting before bulk led schematic symbol change
Parts:
- D1, D11, D129, D13, D132, D134, D136, D140, D142, D144, D146, D148, D15, D150, D152, D154, D156, D3, D33, D35, D37, D39, D41, D43, D5, D7, D9: symbol LED_RABG -> LED_RAGB
Connections:
- net at D1.3 (GK), D129.3 (GK), D142.3 (GK)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: now also D101.4 (GK), D103.4 (GK), D65.4 (GK), D67.4 (GK), D69.4 (GK), D71.4 (GK), D97.4 (GK), D99.4 (GK), R52.1; no longer D101.3 (BK), D103.3 (BK), D65.3 (BK), D67.3 (BK), D69.3 (BK), D71.3 (BK), D97.3 (BK), D99.3 (BK), R56.1
- net at D1.4 (BK), D129.4 (BK), D142.4 (BK)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: now also D101.3 (BK), D103.3 (BK), D65.3 (BK), D67.3 (BK), D69.3 (BK), D71.3 (BK), D97.3 (BK), D99.3 (BK), R56.1; no longer D101.4 (GK), D103.4 (GK), D65.4 (GK), D67.4 (GK), D69.4 (GK), D71.4 (GK), D97.4 (GK), D99.4 (GK), R52.1
- net at D105.3 (BK), D107.3 (BK), D109.3 (BK)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: now also D11.4 (BK), D13.4 (BK), D132.4 (BK), D146.4 (BK), D148.4 (BK), D15.4 (BK), D41.4 (BK), D43.4 (BK), D9.4 (BK); no longer D11.3 (BK), D13.3 (BK), D132.3 (BK), D146.3 (BK), D148.3 (BK), D15.3 (BK), D41.3 (BK), D43.3 (BK), D9.3 (BK)
- net at D105.4 (GK), D107.4 (GK), D109.4 (GK)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: now also D11.3 (GK), D13.3 (GK), D132.3 (GK), D146.3 (GK), D148.3 (GK), D15.3 (GK), D41.3 (GK), D43.3 (GK), D9.3 (GK); no longer D11.4 (GK), D13.4 (GK), D132.4 (GK), D146.4 (GK), D148.4 (GK), D15.4 (GK), D41.4 (GK), D43.4 (GK), D9.4 (GK)
- net at D113.3 (BK), D115.3 (BK), D117.3 (BK)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: now also D136.4 (BK), D150.4 (BK), D152.4 (BK); no longer D136.3 (BK), D150.3 (BK), D152.3 (BK)
- net at D113.4 (GK), D115.4 (GK), D117.4 (GK)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: now also D136.3 (GK), D150.3 (GK), D152.3 (GK); no longer D136.4 (GK), D150.4 (GK), D152.4 (GK)
- net at D121.3 (BK), D123.3 (BK), D125.3 (BK)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: now also D134.4 (BK), D140.4 (BK), D154.4 (BK), D156.4 (BK); no longer D134.3 (BK), D140.3 (BK), D154.3 (BK), D156.3 (BK)
- net at D121.4 (GK), D123.4 (GK), D125.4 (GK)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: now also D134.3 (GK), D140.3 (GK), D154.3 (GK), D156.3 (GK); no longer D134.4 (GK), D140.4 (GK), D154.4 (GK), D156.4 (GK)
Changed lines of the file:
@@
 $EndComp
 $Comp
-L LED_RABG D1
+L LED_RAGB D1
 U 1 1 5A13025C
 P 8300 3500
@@
 $EndComp
 $Comp
-L LED_RABG D3
+L LED_RAGB D3
 U 1 1 5A132308
 P 9550 3500
@@
 $EndComp
 $Comp
-L LED_RABG D5
+L LED_RAGB D5
 U 1 1 5A132C84
 P 10800 3500
@@
 $EndComp
 $Comp
-L LED_RABG D7
+L LED_RAGB D7
 U 1 1 5A132CA1
 P 12050 3500
@@
 $EndComp
 $Comp
-L LED_RABG D9
+L LED_RAGB D9
 U 1 1 5A1356CD
 P 8300 4550
@@
 $EndComp
 $Comp
-L LED_RABG D11
+L LED_RAGB D11
 U 1 1 5A1356E8
 P 9550 4550
@@
 $EndComp
 $Comp
-L LED_RABG D13
+L LED_RAGB D13
 U 1 1 5A135705
 P 10800 4550
@@
 $EndComp
 $Comp
-L LED_RABG D15
+L LED_RAGB D15
 U 1 1 5A135720
 P 12050 4550
@@
 $EndComp
 $Comp
-L LED_RABG D33
+L LED_RAGB D33
 U 1 1 5A13DCD2
 P 13300 3500
@@
 $EndComp
 $Comp
-L LED_RABG D35
+L LED_RAGB D35
 U 1 1 5A13DCED
 P 14550 3500
@@
 $EndComp
 $Comp
-L LED_RABG D37
+L LED_RAGB D37
 U 1 1 5A13DD0A
 P 15800 3500
@@
 $EndComp
 $Comp
-L LED_RABG D39
+L LED_RAGB D39
 U 1 1 5A13DD25
 P 17050 3500
@@
 $EndComp
 $Comp
-L LED_RABG D41
+L LED_RAGB D41
 U 1 1 5A13DD56
 P 13300 4550
@@
 $EndComp
 $Comp
-L LED_RABG D43
+L LED_RAGB D43
 U 1 1 5A13DD71
 P 14550 4550
@@
 NoConn ~ 9850 13850
 $Comp
-L LED_RABG D129
+L LED_RAGB D129
 U 1 1 5A20E763
 P 18800 3500
@@
 $EndComp
 $Comp
-L LED_RABG D132
+L LED_RAGB D132
 U 1 1 5A20E775
 P 18800 4550
@@
 $EndComp
 $Comp
-L LED_RABG D136
+L LED_RAGB D136
 U 1 1 5A20E787
 P 18800 5600
@@
 $EndComp
 $Comp
-L LED_RABG D140
+L LED_RAGB D140
 U 1 1 5A20E799
 P 18800 6650
@@
 $EndComp
 $Comp
-L LED_RABG D142
+L LED_RAGB D142
 U 1 1 5A20E7AB
 P 18800 7700
@@
 $EndComp
 $Comp
-L LED_RABG D148
+L LED_RAGB D148
 U 1 1 5A20E7BD
 P 18800 8750
@@
 $EndComp
 $Comp
-L LED_RABG D150
+L LED_RAGB D150
 U 1 1 5A20E7CF
 P 18800 9800
@@
 $EndComp
 $Comp
-L LED_RABG D156
+L LED_RAGB D156
 U 1 1 5A20E7E1
 P 18800 10850
@@
 $EndComp
 $Comp
-L LED_RABG D134
+L LED_RAGB D134
 U 1 1 5A26ABA3
 P 20650 4550
@@
 $EndComp
 $Comp
-L LED_RABG D144
+L LED_RAGB D144
 U 1 1 5A287387
 P 20050 7700
@@
 $EndComp
 $Comp
-L LED_RABG D152
+L LED_RAGB D152
 U 1 1 5A287393
 P 20050 9800
@@
 $EndComp
 $Comp
-L LED_RABG D146
+L LED_RAGB D146
 U 1 1 5A28CB5F
 P 21300 7700
@@
 $EndComp
 $Comp
-L LED_RABG D154
+L LED_RAGB D154
 U 1 1 5A28CB6B
 P 21300 9800

Commit message: successfuly changed component symbols and net names, further developed pcb
Parts:
- D1, D11, D129, D13, D132, D134, D136, D140, D142, D144, D146, D148, D15, D150, D152, D154, D156, D3, D33, D35, D37, D39, D41, D43, D5, D7, D9: value LED_RABG -> LED_RAGB
- D101, D103, D105, D107, D109, D111, D113, D115, D117, D119, D121, D123, D125, D127, D17, D19, D21, D23, D25, D27, D29, D31, D45, D47, D49, D51, D53, D55, D57, D59, D61, D63, D65, D67, D69, D71, D73, D75, D77, D79, D81, D83, D85, D87, D89, D91, D93, D95, D97, D99: value LED_RABG -> LED_RAGB; symbol LED_RABG -> LED_RAGB
Connections:
- net PWM_BLUE1: now also Q28.1 (G), R28.1; no longer Q32.1 (G), R32.1
- net PWM_BLUE2: now also Q27.1 (G), R27.1; no longer Q31.1 (G), R31.1
- net PWM_BLUE3: now also Q26.1 (G), R26.1; no longer Q30.1 (G), R30.1
- net PWM_BLUE4: now also Q25.1 (G), R25.1; no longer Q29.1 (G), R29.1
- net PWM_GREEN1: now also Q32.1 (G), R32.1; no longer Q28.1 (G), R28.1
- net PWM_GREEN2: now also Q31.1 (G), R31.1; no longer Q27.1 (G), R27.1
- net PWM_GREEN3: now also Q30.1 (G), R30.1; no longer Q26.1 (G), R26.1
- net PWM_GREEN4: now also Q29.1 (G), R29.1; no longer Q25.1 (G), R25.1
- net at D1.3 (GK), D129.3 (GK), D142.3 (GK)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: now also D101.3 (GK), D103.3 (GK), D65.3 (GK), D67.3 (GK), D69.3 (GK), D71.3 (GK), D97.3 (GK), D99.3 (GK), R56.1; no longer D101.4 (GK), D103.4 (GK), D65.4 (GK), D67.4 (GK), D69.4 (GK), D71.4 (GK), D97.4 (GK), D99.4 (GK), R52.1
- net at D1.4 (BK), D129.4 (BK), D142.4 (BK)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: now also D101.4 (BK), D103.4 (BK), D65.4 (BK), D67.4 (BK), D69.4 (BK), D71.4 (BK), D97.4 (BK), D99.4 (BK), R52.1; no longer D101.3 (BK), D103.3 (BK), D65.3 (BK), D67.3 (BK), D69.3 (BK), D71.3 (BK), D97.3 (BK), D99.3 (BK), R56.1
- net at D105.4 (BK), D107.4 (BK), D109.4 (BK)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: now also D11.4 (BK), D13.4 (BK), D132.4 (BK), D146.4 (BK), D148.4 (BK), D15.4 (BK), D41.4 (BK), D43.4 (BK), D9.4 (BK); no longer D11.3 (GK), D13.3 (GK), D132.3 (GK), D146.3 (GK), D148.3 (GK), D15.3 (GK), D41.3 (GK), D43.3 (GK), D9.3 (GK)
- net at D105.3 (GK), D107.3 (GK), D109.3 (GK)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: now also D11.3 (GK), D13.3 (GK), D132.3 (GK), D146.3 (GK), D148.3 (GK), D15.3 (GK), D41.3 (GK), D43.3 (GK), D9.3 (GK); no longer D11.4 (BK), D13.4 (BK), D132.4 (BK), D146.4 (BK), D148.4 (BK), D15.4 (BK), D41.4 (BK), D43.4 (BK), D9.4 (BK)
- net at D113.3 (GK), D115.3 (GK), D117.3 (GK)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: now also D136.3 (GK), D150.3 (GK), D152.3 (GK); no longer D136.4 (BK), D150.4 (BK), D152.4 (BK)
- net at D113.4 (BK), D115.4 (BK), D117.4 (BK)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: now also D136.4 (BK), D150.4 (BK), D152.4 (BK); no longer D136.3 (GK), D150.3 (GK), D152.3 (GK)
- net at D121.3 (GK), D123.3 (GK), D125.3 (GK)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: now also D134.3 (GK), D140.3 (GK), D154.3 (GK), D156.3 (GK); no longer D134.4 (BK), D140.4 (BK), D154.4 (BK), D156.4 (BK)
- net at D121.4 (BK), D123.4 (BK), D125.4 (BK)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: now also D134.4 (BK), D140.4 (BK), D154.4 (BK), D156.4 (BK); no longer D134.3 (GK), D140.3 (GK), D154.3 (GK), D156.3 (GK)
Other:
- moved on the sheet: Q25, Q26, Q27, Q28, Q29, Q30, Q31, Q32, R25, R26, R27, R28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

Commit message: added logos to pcb
Connections:
- net GRID_BUTTON1: now also D131.1 (K); no longer D139.1 (K)
- net GRID_BUTTON4: now also D139.1 (K); no longer D131.1 (K)
- net K_RED4: now reaches D1.1 (RK), D101.1 (RK), D103.1 (RK), D129.1 (RK), D142.1 (RK), D144.1 (RK), D3.1 (RK), D33.1 (RK), D35.1 (RK), D37.1 (RK), D39.1 (RK), D5.1 (RK), D65.1 (RK), D67.1 (RK), D69.1 (RK), D7.1 (RK), D71.1 (RK), D97.1 (RK), D99.1 (RK), R48.1
- net K_GREEN4: now reaches D1.3 (GK), D101.3 (GK), D103.3 (GK), D129.3 (GK), D142.3 (GK), D144.3 (GK), D3.3 (GK), D33.3 (GK), D35.3 (GK), D37.3 (GK), D39.3 (GK), D5.3 (GK), D65.3 (GK), D67.3 (GK), D69.3 (GK), D7.3 (GK), D71.3 (GK), D97.3 (GK), D99.3 (GK), R56.1
- net K_BLUE4: now reaches D1.4 (BK), D101.4 (BK), D103.4 (BK), D129.4 (BK), D142.4 (BK), D144.4 (BK), D3.4 (BK), D33.4 (BK), D35.4 (BK), D37.4 (BK), D39.4 (BK), D5.4 (BK), D65.4 (BK), D67.4 (BK), D69.4 (BK), D7.4 (BK), D71.4 (BK), D97.4 (BK), D99.4 (BK), R52.1
- net K_RED3: now reaches D105.1 (RK), D107.1 (RK), D109.1 (RK), D11.1 (RK), D111.1 (RK), D13.1 (RK), D132.1 (RK), D146.1 (RK), D148.1 (RK), D15.1 (RK), D41.1 (RK), D43.1 (RK), D45.1 (RK), D47.1 (RK), D73.1 (RK), D75.1 (RK), D77.1 (RK), D79.1 (RK), D9.1 (RK), R49.1
- net K_GREEN3: now reaches D105.3 (GK), D107.3 (GK), D109.3 (GK), D11.3 (GK), D111.3 (GK), D13.3 (GK), D132.3 (GK), D146.3 (GK), D148.3 (GK), D15.3 (GK), D41.3 (GK), D43.3 (GK), D45.3 (GK), D47.3 (GK), D73.3 (GK), D75.3 (GK), D77.3 (GK), D79.3 (GK), D9.3 (GK), R57.1
- net K_BLUE3: now reaches D105.4 (BK), D107.4 (BK), D109.4 (BK), D11.4 (BK), D111.4 (BK), D13.4 (BK), D132.4 (BK), D146.4 (BK), D148.4 (BK), D15.4 (BK), D41.4 (BK), D43.4 (BK), D45.4 (BK), D47.4 (BK), D73.4 (BK), D75.4 (BK), D77.4 (BK), D79.4 (BK), D9.4 (BK), R53.1
- net K_RED2: now reaches D113.1 (RK), D115.1 (RK), D117.1 (RK), D119.1 (RK), D136.1 (RK), D150.1 (RK), D152.1 (RK), D17.1 (RK), D19.1 (RK), D21.1 (RK), D23.1 (RK), D49.1 (RK), D51.1 (RK), D53.1 (RK), D55.1 (RK), D81.1 (RK), D83.1 (RK), D85.1 (RK), D87.1 (RK), R50.1
- net K_GREEN2: now reaches D113.3 (GK), D115.3 (GK), D117.3 (GK), D119.3 (GK), D136.3 (GK), D150.3 (GK), D152.3 (GK), D17.3 (GK), D19.3 (GK), D21.3 (GK), D23.3 (GK), D49.3 (GK), D51.3 (GK), D53.3 (GK), D55.3 (GK), D81.3 (GK), D83.3 (GK), D85.3 (GK), D87.3 (GK), R58.1
- net K_BLUE2: now reaches D113.4 (BK), D115.4 (BK), D117.4 (BK), D119.4 (BK), D136.4 (BK), D150.4 (BK), D152.4 (BK), D17.4 (BK), D19.4 (BK), D21.4 (BK), D23.4 (BK), D49.4 (BK), D51.4 (BK), D53.4 (BK), D55.4 (BK), D81.4 (BK), D83.4 (BK), D85.4 (BK), D87.4 (BK), R54.1
- net K_RED1: now reaches D121.1 (RK), D123.1 (RK), D125.1 (RK), D127.1 (RK), D134.1 (RK), D140.1 (RK), D154.1 (RK), D156.1 (RK), D25.1 (RK), D27.1 (RK), D29.1 (RK), D31.1 (RK), D57.1 (RK), D59.1 (RK), D61.1 (RK), D63.1 (RK), D89.1 (RK), D91.1 (RK), D93.1 (RK), D95.1 (RK), R51.1
- net K_GREEN1: now reaches D121.3 (GK), D123.3 (GK), D125.3 (GK), D127.3 (GK), D134.3 (GK), D140.3 (GK), D154.3 (GK), D156.3 (GK), D25.3 (GK), D27.3 (GK), D29.3 (GK), D31.3 (GK), D57.3 (GK), D59.3 (GK), D61.3 (GK), D63.3 (GK), D89.3 (GK), D91.3 (GK), D93.3 (GK), D95.3 (GK), R59.1
- net K_BLUE1: now reaches D121.4 (BK), D123.4 (BK), D125.4 (BK), D127.4 (BK), D134.4 (BK), D140.4 (BK), D154.4 (BK), D156.4 (BK), D25.4 (BK), D27.4 (BK), D29.4 (BK), D31.4 (BK), D57.4 (BK), D59.4 (BK), D61.4 (BK), D63.4 (BK), D89.4 (BK), D91.4 (BK), D93.4 (BK), D95.4 (BK), R55.1
- net at D134.2 (A), Q20.3 (D), SW11.1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: now also SW9.1; no longer SW9.2
- net at D135.2 (A): now also SW9.2; no longer SW9.1
Other:
- moved on the sheet: D131, D139, SW6
Changed lines of the file:
@@
 L LL4148 D131
 U 1 1 5A26AB9D
-P 21200 3900
-F 0 "D131" H 21200 4000 50  0000 C CNN
-F 1 "LL4148" H 21200 3800 50  0000 C CNN
-F 2 "Diodes_SMD:D_MiniMELF" H 21200 3725 50  0001 C CNN
-F 3 "" H 21200 3900 50  0001 C CNN
-	1    21200 3900
-	0    -1   -1   0
+P 21350 3900
+F 0 "D131" H 21350 3800 50  0000 C CNN
+F 1 "LL4148" H 21350 4000 50  0000 C CNN
+F 2 "Diodes_SMD:D_MiniMELF" H 21350 3725 50  0001 C CNN
+F 3 "" H 21350 3900 50  0001 C CNN
+	1    21350 3900
+	-1   0    0    1
 $EndComp
 $Comp
@@
 L LL4148 D139
 U 1 1 5A26ABC7
-P 21200 5600
-F 0 "D139" H 21200 5700 50  0000 C CNN
-F 1 "LL4148" H 21200 5500 50  0000 C CNN
-F 2 "Diodes_SMD:D_MiniMELF" H 21200 5425 50  0001 C CNN
-F 3 "" H 21200 5600 50  0001 C CNN
-	1    21200 5600
-	0    -1   -1   0
+P 21350 5350
+F 0 "D139" H 21350 5250 50  0000 C CNN
+F 1 "LL4148" H 21350 5450 50  0000 C CNN
+F 2 "Diodes_SMD:D_MiniMELF" H 21350 5175 50  0001 C CNN
+F 3 "" H 21350 5350 50  0001 C CNN
+	1    21350 5350
+	-1   0    0    1
 $EndComp
 $Comp
@@
 U 1 1 5A26ABE5
 P 21200 4550
-F 0 "SW9" V 21350 4350 50  0000 L CNN
+F 0 "SW9" V 21050 4350 50  0000 L CNN
 F 1 "SW_Push" H 21200 4490 50  0001 C CNN
 F 2 "ProjectLib:Tactile_switch_12x12_black_cap_no_holes" H 21200 4750 50  0001 C CNN
 F 3 "" H 21200 4750 50  0001 C CNN
 	1    21200 4550
-	0    -1   -1   0
+	0    -1   1    0
 $EndComp
 $Comp
@@
 Connection ~ 12050 3250
 Wire Wire Line
-	6050 4100 21200 4100
+	6050 4100 21500 4100
 Connection ~ 11300 4100
 Connection ~ 10050 4100
@@
 Connection ~ 12050 6400
 Wire Wire Line
-	5750 7250 21200 7250
+	5750 7250 21600 7250
 Connection ~ 11300 7250
 Connection ~ 10050 7250
@@
 L SW_Push SW6
 U 1 1 5A2ED1C1
-P 20650 3700
-F 0 "SW6" H 20700 3800 50  0000 L CNN
-F 1 "SW_Push" H 20650 3640 50  0001 C CNN
-F 2 "ProjectLib:Tactile_switch_12x12_black_cap_no_holes" H 20650 3900 50  0001 C CNN
-F 3 "" H 20650 3900 50  0001 C CNN
-	1    20650 3700
+P 20650 3900
+F 0 "SW6" H 20700 4000 50  0000 L CNN
+F 1 "SW_Push" H 20650 3840 50  0001 C CNN
+F 2 "ProjectLib:Tactile_switch_12x12_black_cap_no_holes" H 20650 4100 50  0001 C CNN
+F 3 "" H 20650 4100 50  0001 C CNN
+	1    20650 3900
 	1    0    0    -1
 $EndComp
@@
 Wire Wire Line
 	20050 4300 21200 4300
-Wire Wire Line
-	21200 4100 21200 4050
 Connection ~ 19300 4100
 Wire Wire Line
-	20850 3700 21200 3700
+	20850 3900 21200 3900
 Wire Wire Line
 	20050 2950 20050 4350
@@
 Wire Wire Line
 	20150 5350 20450 5350
-Wire Wire Line
-	21200 7250 21200 5750
 Connection ~ 19300 7250
 Wire Wire Line
 	20850 5350 21200 5350
 Wire Wire Line
-	21200 5350 21200 5450
-Wire Wire Line
 	20050 4750 20050 5450
 Wire Wire Line
@@
 Connection ~ 19750 2550
 Wire Wire Line
-	20450 3700 20050 3700
-Connection ~ 20050 3700
+	20450 3900 20050 3900
+Connection ~ 20050 3900
 $Comp
 L SW_Push SW12
@@
 COLUMN[1..6]
 Wire Wire Line
-	21200 3700 21200 3750
-Wire Wire Line
 	21200 5150 21200 5100
 Wire Wire Line
@@
 $EndComp
 Connection ~ 6050 4400
+Text Label 5000 5650 0    60   ~ 0
+K_RED1
+Text Label 5000 5550 0    60   ~ 0
+K_RED2
+Text Label 5000 5450 0    60   ~ 0
+K_RED3
+Text Label 5000 5350 0    60   ~ 0
+K_RED4
+Text Label 5000 7450 0    60   ~ 0
+K_GREEN4
+Text Label 5000 7550 0    60   ~ 0
+K_GREEN3
+Text Label 5000 7650 0    60   ~ 0
+K_GREEN2
+Text Label 5000 7750 0    60   ~ 0
+K_GREEN1
+Text Label 5000 9850 0    60   ~ 0
+K_BLUE1
+Text Label 5000 9750 0    60   ~ 0
+K_BLUE2
+Text Label 5000 9650 0    60   ~ 0
+K_BLUE3
+Text Label 5000 9550 0    60   ~ 0
+K_BLUE4
+Wire Wire Line
+	21500 4100 21500 5350
+Wire Wire Line
+	21600 7250 21600 3900
+Wire Wire Line
+	21600 3900 21500 3900
 $EndSCHEMATC
