File: midi_grid.kicad_pcb (KiCad board)
At the start: 2 copper layers, 275 x 200 mm, 313 parts, among them J1 USB_OTG, J2 3.5mm jack, J3 3.5mm jack, J4 Conn_01x04_Male, Q1 BSS83P, Q10 BSS83P, Q11 BSS83P, Q12 BSS83P, Q13 BSS83P, Q14 BSS83P, Q15 BSS83P, Q16 BSS83P, Q17 BSS83P, Q18 BSS83P, Q19 BSS83P, Q2 BSS83P, Q20 BSS83P, Q21 NX7002AK, Q22 NX7002AK, Q23 NX7002AK, Q24 NX7002AK, Q25 NX7002AK, Q26 NX7002AK, Q27 NX7002AK, Q28 NX7002AK, Q29 NX7002AK, Q3 BSS83P, Q30 NX7002AK, Q31 NX7002AK, Q32 NX7002AK, Q33 NX7002AK, Q34 NX7002AK, Q4 BSS83P, Q5 BSS83P, Q6 BSS83P, Q7 BSS83P, Q8 BSS83P, Q9 BSS83P, SW1 Button_matrix_4x4, SW10 SW_Push, SW11 SW_Push, SW12 SW_Push, SW13 SW_Push, SW14 SW_Push, SW15 SW_Push, SW16 SW_Push, SW17 SW_Push, SW18 SW_Push, SW19 SW_Push, SW2 Button_matrix_4x4, SW20 SW_Push, SW21 SW_Push, SW22 SW_Push, SW23 SW_Push, SW24 SW_Push, SW25 EC12E24204A9, SW26 EC12E24204A9, SW3 Button_matrix_4x4, SW4 Button_matrix_4x4, SW5 SW_Push, SW6 SW_Push, SW7 SW_Push, SW8 SW_Push, SW9 SW_Push, U1 74HC138, U2 74HC138, U3 74HC138, U4 USBUF, U5 STM32F411RCT6, U6 LD1117STR, U7 LTV-357T, Y1 8MHz

Commit message: added logos to pcb
Parts:
- added SW66: SW_DIP_x01, ProjectLib:Logo_OSHW, B.Cu at (115.5, 217.5)
- added SW69: SW_DIP_x01, ProjectLib:qr_url, B.Cu at (90.5, 213.5)
- C4: moved to B.Cu
- moved TP6 230.7 mm to (345.5, 76.5)
- moved TP1 230.5 mm to (354.0, 112.0)
- moved TP2 215.1 mm to (353.0, 123.5)
- moved TP3 214.5 mm to (353.5, 118.5)
- moved C4 183.1 mm to (309.5, 85.5), turned to 180 degrees
- moved C5 174.4 mm to (347.0, 127.5)
- moved D131 16.8 mm to (320.5, 112.5)
- moved D139 13.8 mm to (306.5, 125.5)
- moved R48 8.63 mm to (268.0, 80.5)
- moved R49 8.63 mm to (268.0, 83.0)
- moved U7 7.02 mm to (308.0, 59.0)
- moved R45 7.00 mm to (312.0, 64.0)
- moved R24 4.74 mm to (274.5, 91.5)
- moved D158 4.53 mm to (305.5, 52.0)
- moved R46 4.53 mm to (309.5, 52.0), turned to 90 degrees
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Connections:
- net Net-(D1-Pad1) renamed /grid/K_RED4
- net Net-(D1-Pad3) renamed /grid/K_GREEN4
- net Net-(D1-Pad4) renamed /grid/K_BLUE4
- net Net-(D105-Pad1) renamed /grid/K_RED3
- net Net-(D105-Pad3) renamed /grid/K_GREEN3
- net Net-(D105-Pad4) renamed /grid/K_BLUE3
- net Net-(D113-Pad1) renamed /grid/K_RED2
- net Net-(D113-Pad3) renamed /grid/K_GREEN2
- net Net-(D113-Pad4) renamed /grid/K_BLUE2
- net Net-(D121-Pad1) renamed /grid/K_RED1
- net Net-(D121-Pad3) renamed /grid/K_GREEN1
- net Net-(D121-Pad4) renamed /grid/K_BLUE1
- D131 pad 1: /grid/GRID_BUTTON4 -> /grid/GRID_BUTTON1
- D139 pad 1: /grid/GRID_BUTTON1 -> /grid/GRID_BUTTON4
- SW9 pad 1: Net-(D135-Pad2) -> Net-(D134-Pad2)
- SW9 pad 2: Net-(D134-Pad2) -> Net-(D135-Pad2)
- U5 pad 20: /mcu/COL4 -> /mcu/COL5
- U5 pad 21: /mcu/COL5 -> /mcu/COL4
Routing:
- net /grid/GRID_BUTTON1: track 620.8 -> 864.6 mm, vias 5 -> 6
- net /grid/GRID_BUTTON2: track 587.2 -> 794.5 mm, vias 5 -> 6
- net /grid/GRID_BUTTON3: track 607.4 -> 785.3 mm, vias 5 -> 6
- net /grid/GRID_BUTTON4: track 570.0 -> 744.2 mm, vias 5 -> 6
- net /digital_io/ROTARY1_B: track 4.13 -> 121.6 mm, vias 0 -> 1
- net /digital_io/ROTARY1_A: track 3.71 -> 119.3 mm, vias 0 -> 1
- net /mcu/COL2: track 8.68 -> 122.5 mm, vias 0 -> 4
- net /mcu/COL1: track 8.32 -> 118.1 mm, vias 0 -> 4
- net /mcu/COL4: track 0.00 -> 100.7 mm, vias 0 -> 4
- net /digital_io/BUTTON1: track 3.05 -> 100.0 mm, vias 0 -> 1
- net /digital_io/ROTARY2_B: track 0.00 -> 82.1 mm
- net /digital_io/ROTARY2_A: track 0.00 -> 80.7 mm
- net /digital_io/BUTTON2: track 0.00 -> 62.2 mm
- net /mcu/COL3: track 63.8 -> 124.7 mm, vias 1 -> 4
- net /mcu/COL5: track 0.00 -> 47.8 mm, vias 0 -> 2
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
Commit message: added net names in grid schematic
Parts:
- moved SW69 150.0 mm to (240.5, 214.0)
- moved U3 112.9 mm to (278.2, 136.0), turned to 0 degrees
- moved SW66 50.0 mm to (165.5, 216.8)
- moved Q18 40.9 mm to (362.2, 143.0)
- moved R18 40.9 mm to (359.8, 143.0)
- moved J4 3.16 mm to (335.5, 96.0)
- moved D114 1.00 mm to (179.0, 205.5), turned to 180 degrees
- moved D116 1.00 mm to (204.0, 205.5), turned to 180 degrees
- moved D118 1.00 mm to (229.0, 205.5), turned to 180 degrees
Connections:
- Q17 pad 1: Net-(Q17-Pad1) -> /grid/G17
- Q18 pad 1: Net-(Q18-Pad1) -> /grid/G18
- Q19 pad 1: Net-(Q19-Pad1) -> /grid/G19
- Q20 pad 1: Net-(Q20-Pad1) -> /grid/G20
- R17 pad 2: Net-(Q17-Pad1) -> /grid/G17
- R18 pad 2: Net-(Q18-Pad1) -> /grid/G18
- R19 pad 2: Net-(Q19-Pad1) -> /grid/G19
- R20 pad 2: Net-(Q20-Pad1) -> /grid/G20
- U3 pad 12: Net-(U3-Pad12) -> /grid/G20
- U3 pad 13: Net-(U3-Pad13) -> /grid/G19
Routing:
- net /mcu/COL6: track 0.00 -> 29.5 mm, vias 0 -> 1
- net /mcu/SWDCLK: track 0.00 -> 25.9 mm
- net +3V3: track 47.0 -> 67.8 mm
- net /mcu/SWDIO: track 9.46 -> 27.8 mm
- net /grid/GRID_BUTTON2: track 794.5 -> 800.3 mm
- net GND: track 54.7 -> 58.7 mm, vias 2 -> 4
- net /mcu/COL5: track 47.8 -> 45.0 mm, vias 2 -> 1
- net Net-(D118-Pad2): track 3.15 -> 4.50 mm
- net Net-(D116-Pad2): track 3.15 -> 4.50 mm
- net Net-(D114-Pad2): track 3.15 -> 4.50 mm
- net /mcu/COL2: track 122.5 -> 123.8 mm
- net /mcu/COL3: track 124.7 -> 126.0 mm
- net /mcu/COL1: track 118.1 -> 118.9 mm
- net Net-(D88-Pad2): track 3.15 -> 2.40 mm
- net (no net): vias 1 -> 2
Other:
- board text added: "Designed by Gediminas Žukaitis Version 1.0 github.com/zukaitis/midi-grid Date of revision: 2018-01-25"

Commit message: pcb development
Parts:
- removed SW66: SW_DIP_x01, ProjectLib:Logo_OSHW
- removed SW69: SW_DIP_x01, ProjectLib:qr_url
- added GR1: OSHW logo, ProjectLib:Logo_OSHW, B.Cu at (165.5, 217.0)
- added GR2: QR code, ProjectLib:qr_url, B.Cu at (240.5, 214.2)
- moved Q17 118.0 mm to (287.5, 138.2), turned to 270 degrees
- moved R17 114.2 mm to (287.5, 135.8), turned to 180 degrees
- moved C3 113.4 mm to (280.5, 140.8), turned to 180 degrees
- moved Q19 101.6 mm to (294.5, 138.2), turned to 270 degrees
- moved R19 98.3 mm to (294.5, 135.8), turned to 180 degrees
- moved R20 95.2 mm to (298.0, 135.8), turned to 180 degrees
- moved Q20 93.8 mm to (298.0, 138.2), turned to 270 degrees
- moved Q18 71.4 mm to (291.0, 138.2), turned to 270 degrees
- moved R18 69.1 mm to (291.0, 135.8), turned to 180 degrees
- moved U3 1.03 mm to (278.0, 137.0)
Routing:
- net /mcu/COL6: track 29.5 -> 98.5 mm, vias 1 -> 4
- net +5V: track 277.7 -> 329.2 mm, vias 4 -> 5
- net Net-(D129-Pad2): track 95.2 -> 117.9 mm, vias 0 -> 1
- net Net-(D144-Pad2): track 106.4 -> 124.8 mm, vias 0 -> 2
- net /mcu/COL1: track 118.9 -> 124.1 mm, vias 4 -> 5
- net /mcu/COL2: track 123.8 -> 128.8 mm, vias 4 -> 5
- net /mcu/COL3: track 126.0 -> 130.8 mm, vias 4 -> 5
- net Net-(D142-Pad2): track 95.6 -> 100.1 mm, vias 0 -> 1
- net /mcu/COL5: track 45.0 -> 48.4 mm, vias 1 -> 2
- net +3V3: track 67.8 -> 70.4 mm
- net /grid/G17: track 0.00 -> 1.58 mm
- net /grid/G20: track 0.00 -> 1.58 mm
- net /grid/G19: track 0.00 -> 1.58 mm
- net /grid/G18: track 0.00 -> 1.58 mm
- net /mcu/COL4: track 100.7 -> 101.7 mm
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