File: Hardware/midi_grid.kicad_pcb (KiCad board)
At the start: 2 copper layers, 275 x 200 mm, 328 parts, among them J1 USB_OTG, J2 3.5mm jack, J3 3.5mm jack, J4 Conn_01x04_Male, M1 Mounting_hole, M2 Mounting_hole, M3 Mounting_hole, Q1 BSH205G2, Q10 BSH205G2, Q11 BSH205G2, Q12 BSH205G2, Q13 BSH205G2, Q14 BSH205G2, Q15 BSH205G2, Q16 BSH205G2, Q17 BSH205G2, Q18 BSH205G2, Q19 BSH205G2, Q2 BSH205G2, Q20 BSH205G2, Q21 NX7002AK, Q22 NX7002AK, Q23 NX7002AK, Q24 NX7002AK, Q25 NX7002AK, Q26 NX7002AK, Q27 NX7002AK, Q28 NX7002AK, Q29 NX7002AK, Q3 BSH205G2, Q30 NX7002AK, Q31 NX7002AK, Q32 NX7002AK, Q33 NX7002AK, Q34 NX7002AK, Q4 BSH205G2, Q5 BSH205G2, Q6 BSH205G2, Q7 BSH205G2, Q8 BSH205G2, Q9 BSH205G2, SW1 Button_matrix_4x4, SW10 SW_Push, SW11 SW_Push, SW12 SW_Push, SW13 SW_Push, SW14 SW_Push, SW15 SW_Push, SW16 SW_Push, SW17 SW_Push, SW18 SW_Push, SW19 SW_Push, SW2 Button_matrix_4x4, SW20 SW_Push, SW21 SW_Push, SW22 SW_Push, SW23 SW_Push, SW24 SW_Push, SW25 EC12E24204A9, SW26 EC12E24204A9, SW3 Button_matrix_4x4, SW4 Button_matrix_4x4, SW5 SW_Push, SW6 SW_Push, SW7 SW_Push, SW8 SW_Push, SW9 SW_Push, U1 STM32F411RCT6, U2 74HC138, U3 74HC138, U4 74HC138, U5 USBUF02W6, U6 VO617A, U7 LD1117STR, Y1 8MHz

Commit message: replaced all models with .step, deleted .wrl models
Parts:
- SW10, SW12, SW13, SW14, SW15, SW16, SW17, SW18, SW19, SW20, SW23, SW5, SW7: footprint project_library:Tactile_switch_12x12_black_cap -> project_library:Tactile_switch_12x12
- SW11, SW6, SW8, SW9: footprint project_library:Tactile_switch_12x12_black_cap_no_holes -> project_library:Tactile_switch_12x12_no_holes
- SW24: footprint project_library:Tactile_switch_12x12_red_cap -> project_library:Tactile_switch_12x12
