File: Hardware/psu.sch (KiCad schematic (older format))
At the start: 10 parts, among them U7 LD1117STR

Commit message: linked footprints with 3D models in project directory
Parts:
- F1: Catalog link (none) -> https://eu.mouser.com/productdetail/?qs=PWhpLWeW8wckT8hV5jL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
- U7: Catalog link (none) -> http://uk.farnell.com/stmicroelectronics/ld1117str/ic-v-reg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
Changed lines of the file:
@@
 F 2 "project_library:R_1206" H 4750 3500 50  0001 L CNN
 F 3 "" H 4700 3700 50  0001 C CNN
+F 4 "https://eu.mouser.com/productdetail/?qs=PWhpLWeW8wckT8hV5jLiAA%3D%3D" V 4700 3700 60  0001 C CNN "Catalog link"
 	1    4700 3700
 	0    1    1    0
@@
 F 2 "project_library:SOT-223-3Lead_TabPin2" H 5950 3700 50  0001 C CNN
 F 3 "" H 5950 3700 50  0001 C CNN
+F 4 "http://uk.farnell.com/stmicroelectronics/ld1117str/ic-v-reg-adj-1-25-15v-smd-1117/dp/1202824" H 5950 3700 60  0001 C CNN "Catalog link"
 	1    5950 3700
 	1    0    0    -1

Commit message: converted all components except big tactile switches
Parts:
- C16, C17, C18, C19, C20, C21: symbol C_Small -> project_library:C_Small
- F1: symbol Polyfuse -> project_library:Polyfuse
- R64, R65: symbol R -> project_library:R
- U7: symbol LM1117-ADJ -> project_library:LM1117-ADJ
Changed lines of the file:
@@
-EESchema Schematic File Version 2
-LIBS:project_library
-LIBS:power
-LIBS:device
-LIBS:switches
-LIBS:relays
-LIBS:motors
-LIBS:transistors
-LIBS:conn
-LIBS:linear
-LIBS:regul
-LIBS:74xx
-LIBS:cmos4000
-LIBS:adc-dac
-LIBS:memory
-LIBS:xilinx
-LIBS:microcontrollers
-LIBS:diode
-LIBS:dsp
-LIBS:microchip
-LIBS:analog_switches
-LIBS:motorola
-LIBS:texas
-LIBS:intel
-LIBS:audio
-LIBS:interface
-LIBS:digital-audio
-LIBS:philips
-LIBS:display
-LIBS:cypress
-LIBS:siliconi
-LIBS:opto
-LIBS:atmel
-LIBS:contrib
-LIBS:valves
-LIBS:stm32
-LIBS:ESD_Protection
+EESchema Schematic File Version 4
 LIBS:midi_grid-cache
-EELAYER 25 0
+EELAYER 30 0
 EELAYER END
 $Descr A4 11693 8268
@@
 $EndDescr
 $Comp
-L C_Small C17
+L project_library:C_Small C17
 U 1 1 5A21CDC2
 P 5350 3900
@@
 $EndComp
 $Comp
-L +3.3V #PWR0137
+L project_library:+3.3V #PWR0137
 U 1 1 5A21CDCF
 P 7150 3600
@@
 $EndComp
 $Comp
-L GND #PWR0138
+L project_library:GND #PWR0138
 U 1 1 5A21CF18
 P 5350 4100
@@
 	5350 3700 5350 3800
 $Comp
-L C_Small C16
+L project_library:C_Small C16
 U 1 1 5A21CF38
 P 4950 3900
@@
 Connection ~ 5350 3700
 $Comp
-L GND #PWR0139
+L project_library:GND #PWR0139
 U 1 1 5A21CF81
 P 4950 4100
@@
 	4950 4000 4950 4100
 $Comp
-L C_Small C18
+L project_library:C_Small C18
 U 1 1 5A21D03A
 P 6750 3900
@@
 	6750 3700 6750 3800
 $Comp
-L GND #PWR0140
+L project_library:GND #PWR0140
 U 1 1 5A21D041
 P 6750 4100
@@
 	6750 4000 6750 4100
 $Comp
-L C_Small C19
+L project_library:C_Small C19
 U 1 1 5A21D0A4
 P 7150 3900
@@
 	7150 3600 7150 3800
 $Comp
-L GND #PWR0141
+L project_library:GND #PWR0141
 U 1 1 5A21D0AB
 P 7150 4100
@@
 Connection ~ 6750 3700
 $Comp
-L R R64
+L project_library:R R64
 U 1 1 5A220887
 P 6350 3900
@@
 $EndComp
 $Comp
-L R R65
+L project_library:R R65
 U 1 1 5A2211BF
 P 5950 4300
@@
 $EndComp
 $Comp
-L GND #PWR0142
+L project_library:GND #PWR0142
 U 1 1 5A221A3F
 P 5950 4500
@@
 Vin
 $Comp
-L Polyfuse F1
+L project_library:Polyfuse F1
 U 1 1 5A33C036
 P 4700 3700
@@
 	4450 3700 4550 3700
 $Comp
-L LM1117-ADJ U7
+L project_library:LM1117-ADJ U7
 U 1 1 5A32EC50
 P 5950 3700
@@
 Connection ~ 6350 3700
 $Comp
-L +5V #PWR0143
+L project_library:+5V #PWR0143
 U 1 1 5A43721A
 P 4950 3600
@@
 $EndComp
 $Comp
-L C_Small C21
+L project_library:C_Small C21
 U 1 1 5A73B3AD
 P 5350 4700
@@
 $EndComp
 $Comp
-L +5V #PWR0144
+L project_library:+5V #PWR0144
 U 1 1 5A73B4E2
 P 5350 4600
@@
 $EndComp
 $Comp
-L GND #PWR0145
+L project_library:GND #PWR0145
 U 1 1 5A73B508
 P 5350 4850
@@
 $EndComp
 $Comp
-L C_Small C20
+L project_library:C_Small C20
 U 1 1 5A73B65D
 P 4950 4700
@@
 $EndComp
 $Comp
-L +5V #PWR0146
+L project_library:+5V #PWR0146
 U 1 1 5A73B663
 P 4950 4600
@@
 $EndComp
 $Comp
-L GND #PWR0147
+L project_library:GND #PWR0147
 U 1 1 5A73B669
 P 4950 4850
