File: Hardware/lcd_board/lcd_board.kicad_pcb (KiCad board)
At the start: 2 copper layers, 46 x 55.5 mm, 10 parts, among them J1 Conn_01x08_Male, Q1 BSS84

Commit message: commiting hanging changes, dont even remember what they are
Connections:
- LCD1 pad 3: /CS -> /DC
- LCD1 pad 5: /DC -> /CS
Routing:
- net /CS: track 9.38 -> 10.6 mm
- net GND: vias 48 -> 49
