File: Hardware/lcd_board/lcd_board.sch (KiCad schematic (older format))
At the start: 10 parts, among them J1 Conn_01x08_Male, Q1 BSS84

Commit message: commiting hanging changes, dont even remember what they are
Connections:
- net CS: now also LCD1.5 (DC/RS); no longer LCD1.3 (CS)
- net DC: now also LCD1.3 (CS); no longer LCD1.5 (DC/RS)
Changed lines of the file:
@@
 Connection ~ 7200 3700
-Wire Wire Line
-	5650 3300 7300 3300
-Wire Wire Line
-	5650 3200 7300 3200
 Wire Wire Line
 	6950 3500 6950 3100
@@
 	1    0    0    -1
 $EndComp
+Wire Wire Line
+	7300 3200 6750 3200
+Wire Wire Line
+	6750 3200 6750 3300
+Wire Wire Line
+	6750 3300 5650 3300
+Wire Wire Line
+	5650 3200 6650 3200
+Wire Wire Line
+	6650 3200 6650 3000
+Wire Wire Line
+	6650 3000 7150 3000
+Wire Wire Line
+	7150 3000 7150 3300
+Wire Wire Line
+	7150 3300 7300 3300
 $EndSCHEMATC
